Commit message: added fan blade and paint gun to xacro

File: rpi_abb_irb6640_180_255_support/urdf/6640.urdf.xacro (robot description, xacro)
@@ -4,5 +4,7 @@
 <!-- |    EDITING THIS FILE BY HAND IS NOT RECOMMENDED                                 | -->
 <!-- =================================================================================== -->
-<robot name="abb_irb6640_180_255">
+<robot name="abb_irb6640" xmlns:xacro="http://ros.org/wiki/xacro">
+<xacro:macro name="abb_irb6640" params="prefix">
+<!--<robot name="abb_irb6640_180_255">-->
   <!-- link list -->
   <link name="base_link">
@@ -325,3 +327,4 @@
     <child link="base_link"/>
   </joint>
+</xacro:macro>
 </robot>
