Commit message: rviz can launch with tesseract planning model but will crash or error when trying to plan

File: rpi_abb_irb6640_180_255_support/urdf/6640.urdf (robot description, URDF)
Before this commit: robot abb_irb6640_180_255, 0 links, 0 joints
Links:
- added link base
- added link base_link, mass 254.138; collision box size=1.016 .729 .24; visual mesh filename=package://rpi_abb_irb6640_180_255_support/meshes/irb6640_18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
- added link link_1, mass 469.323; collision box size=.31 .528 .368; collision box size=.436 .328 .192
- added link link_2, mass 153.009; collision box size=.251 .169 .058; collision box size=.538 1.429 .311
- added link link_3, mass 212.29; collision box size=.052 .085 .102; collision box size=.052 .109 .102
- added link link_4, mass 185.22; collision box size=.145 .278 .075; collision box size=.145 .278 .092
- added link link_5, mass 26.117; collision cylinder length=.307 radius=.107; visual mesh filename=package://rpi_abb_irb6640_180_255_support/meshes/irb6640_18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
- added link link_6, mass 3.371; collision cylinder length=.037 radius=.109; visual mesh filename=package://rpi_abb_irb6640_180_255_support/meshes/irb6640_18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
- added link tool0
- added link world
Joints:
- added joint base_link-base: type fixed, parent base_link, child base, origin xyz=0 0 0 rpy=0 0 0
- added joint fixed: type fixed, parent world, child base_link
- added joint joint_1: type revolute, parent base_link, child link_1, origin xyz=0 0 0.780 rpy=0 0 0, axis 0 0 1, limit lower=-2.967 upper=2.967 effort=0 velocity=1.7453
- added joint joint_2: type revolute, parent link_1, child link_2, origin xyz=0.320 0 0 rpy=0 0 0, axis 0 1 0, limit lower=-1.134 upper=1.4855 effort=0 velocity=1.5707
- added joint joint_3: type revolute, parent link_2, child link_3, origin xyz=0 0 1.075 rpy=0 0 0, axis 0 1 0, limit lower=-3.142 upper=1.222 effort=0 velocity=1.5707
- added joint joint_4: type revolute, parent link_3, child link_4, origin xyz=0 0 0.2 rpy=0 0 0, axis 1 0 0, limit lower=-5.236 upper=5.236 effort=0 velocity=2.9671
- added joint joint_5: type revolute, parent link_4, child link_5, origin xyz=1.1425 0 0  rpy=0 0 0, axis 0 1 0, limit lower=-2.094 upper=2.094 effort=0 velocity=2.4435
- added joint joint_6: type revolute, parent link_5, child link_6, origin xyz=0.2 0 0  rpy=0 0 0, axis 1 0 0, limit lower=-6.283 upper=6.283 effort=0 velocity=3.3161
- added joint joint_6-tool0: type fixed, parent link_6, child tool0, origin xyz=0 0 0 rpy=0 1.57079632679 0

File: rpi_abb_irb6640_180_255_support/urdf/workcell.xacro (robot description, xacro)
@@ -1,6 +1,6 @@
 <?xml version="1.0" ?>
-<robot name="irb6640" xmlns:xacro="http://ros.org/wiki/xacro">
+<robot name="abb_irb6640_180_255" xmlns:xacro="http://ros.org/wiki/xacro">
   <xacro:include filename="$(find rpi_abb_irb6640_180_255_support)/urdf/6640.urdf.xacro" />
-    <link name="generic_fan_blade">
+<!--    <link name="generic_fan_blade">
       <collision>
         <origin rpy="0 0 0" xyz="1.2 0 0"/>
@@ -27,7 +27,7 @@
         </geometry>
       </visual>
-    </link>
-    <xacro:abb_irb6640 prefix=""/>
-    <joint name="world_to_fan" type="fixed">
+    </link>-->
+    <xacro:abb_irb6640_180_255 prefix=""/>
+<!--    <joint name="world_to_fan" type="fixed">
         <parent link="world"/>
         <child link="generic_fan_blade"/>
@@ -38,4 +38,4 @@
         <child link="paint_gun"/>
         <origin xyz="0 0 0" rpy="0 0 0"/>
-    </joint>
+    </joint>-->
 </robot>
