Commit message: tool path waypoints show up in rviz when planner service is called. planning is failing though

File: rpi_abb_irb6640_180_255_support/urdf/workcell.xacro (robot description, xacro)
@@ -2,5 +2,5 @@
 <robot name="abb_irb6640_180_255" xmlns:xacro="http://ros.org/wiki/xacro">
   <xacro:include filename="$(find rpi_abb_irb6640_180_255_support)/urdf/6640.urdf.xacro" />
-<!--    <link name="generic_fan_blade">
+    <link name="generic_fan_blade">
       <collision>
         <origin rpy="0 0 0" xyz="1.2 0 0"/>
@@ -27,10 +27,10 @@
         </geometry>
       </visual>
-    </link>-->
+    </link>
     <xacro:abb_irb6640_180_255 prefix=""/>
-<!--    <joint name="world_to_fan" type="fixed">
+    <joint name="world_to_fan" type="fixed">
         <parent link="world"/>
         <child link="generic_fan_blade"/>
-        <origin xyz="2.2 0 0" rpy="0 -1.57 0"/>
+        <origin xyz="1.5 -1.1 0.5" rpy="-2.356 0 1.57"/>
     </joint>
     <joint name="tool0_to_gun" type="fixed">
@@ -38,4 +38,4 @@
         <child link="paint_gun"/>
         <origin xyz="0 0 0" rpy="0 0 0"/>
-    </joint>-->
+    </joint>
 </robot>

Commit message: fixed descartes motion planning issue. robot can now follow the waypoints

File: rpi_abb_irb6640_180_255_support/urdf/workcell.xacro (robot description, xacro)
@@ -4,7 +4,7 @@
     <link name="generic_fan_blade">
       <collision>
-        <origin rpy="0 0 0" xyz="1.2 0 0"/>
+        <origin rpy="-1 0 0" xyz="1 0 -.2"/>
         <geometry>
-          <box size="1.016 .729 .24"/>
+          <box size="1.5 .729 .15"/>
         </geometry>
       </collision>
@@ -17,7 +17,7 @@
     <link name="paint_gun">
       <collision>
-        <origin rpy="0 0 0" xyz="0 0 .7"/>
+        <origin rpy="0 0 0" xyz="0 0 .2"/>
         <geometry>
-          <box size="1.016 .729 .24"/>
+          <box size=".2 .2 .2"/>
         </geometry>
       </collision>

Commit message: toolpath is followed by the paint_gun frame instead of tool0 now

File: rpi_abb_irb6640_180_255_support/urdf/workcell.xacro (robot description, xacro)
@@ -17,5 +17,5 @@
     <link name="paint_gun">
       <collision>
-        <origin rpy="0 0 0" xyz="0 0 .2"/>
+        <origin rpy="0 0 0" xyz="0.03 0 -0.3"/>
         <geometry>
           <box size=".2 .2 .2"/>
@@ -23,4 +23,5 @@
       </collision>
       <visual name="visual">
+        <origin rpy="0 0 0" xyz="0.03 0 -0.3"/>
         <geometry>
           <mesh filename="package://rpi_abb_irb6640_180_255_support/meshes/paint_gun.stl" scale="0.001 0.001 0.001"/>
@@ -37,5 +38,5 @@
         <parent link="tool0"/>
         <child link="paint_gun"/>
-        <origin xyz="0 0 0" rpy="0 0 0"/>
+        <origin xyz="-0.03 0 0.3" rpy="0 0 0"/>
     </joint>
 </robot>

Commit message: Kinematics update

File: rpi_abb_irb6640_180_255_support/urdf/workcell.xacro (robot description, xacro)
@@ -1,5 +1,6 @@
 <?xml version="1.0" ?>
 <robot name="abb_irb6640_180_255" xmlns:xacro="http://ros.org/wiki/xacro">
-  <xacro:include filename="$(find rpi_abb_irb6640_180_255_support)/urdf/6640.urdf.xacro" />
+    <xacro:include filename="$(find rpi_abb_irb6640_180_255_support)/urdf/6640.urdf.xacro" />
+    <xacro:abb_irb6640_180_255 prefix=""/>
     <link name="generic_fan_blade">
       <collision>
@@ -17,5 +18,5 @@
     <link name="paint_gun">
       <collision>
-        <origin rpy="0 0 0" xyz="0.03 0 -0.3"/>
+        <origin rpy="0 0 0" xyz="0.0 0 0.0"/>
         <geometry>
           <box size=".2 .2 .2"/>
@@ -23,5 +24,5 @@
       </collision>
       <visual name="visual">
-        <origin rpy="0 0 0" xyz="0.03 0 -0.3"/>
+        <origin rpy="0 0 0" xyz="0.0 0 0.0"/>
         <geometry>
           <mesh filename="package://rpi_abb_irb6640_180_255_support/meshes/paint_gun.stl" scale="0.001 0.001 0.001"/>
@@ -29,5 +30,15 @@
       </visual>
     </link>
-    <xacro:abb_irb6640_180_255 prefix=""/>
+    <joint name="tool0_to_gun" type="fixed">
+        <parent link="tool0"/>
+        <child link="paint_gun"/>
+        <origin xyz="0 0 0" rpy="0 0 0"/>
+    </joint>
+    <link name="paint_tcp"/>
+    <joint name="tool0_to_tcp" type="fixed">
+        <parent link="tool0"/>
+        <child link="paint_tcp"/>
+        <origin xyz="0.075 0 0.4933" rpy="0 0.52359878 0"/>
+    </joint>
     <joint name="world_to_fan" type="fixed">
         <parent link="world"/>
@@ -35,8 +46,3 @@
         <origin xyz="1.5 -1.1 0.5" rpy="-2.356 0 1.57"/>
     </joint>
-    <joint name="tool0_to_gun" type="fixed">
-        <parent link="tool0"/>
-        <child link="paint_gun"/>
-        <origin xyz="-0.03 0 0.3" rpy="0 0 0"/>
-    </joint>
 </robot>
